Commit message: Add base footprint link and joint to akm_base.xacro

File: akm_500_display/urdf/akm_base.xacro (robot description, xacro)
@@ -4,4 +4,11 @@
      For more information, please see http://wiki.ros.org/sw_urdf_exporter -->
 <robot xmlns:xacro="http://www.ros.org/wiki/xacro">
+  <!-- Dummy link as root to work around KDL not supporting inertia on root link -->
+  <link name="base_footprint" />
+  <joint name="base_joint" type="fixed">
+    <origin xyz="0 0 0" rpy="0 0 0" />
+    <parent link="base_footprint" />
+    <child link="base_link" />
+  </joint>
   <link
     name="base_link">
