Commit message: Update wheel names and parameters, remove unused files, and enhance test robot definition

File: akm_500_display/urdf/test_diff_drive.xacro.urdf (robot description, URDF)
Before this commit: robot diff_drive, 4 links, 3 joints
Links:
- added link rear_left_wheel, mass 2; collision sphere radius=0.3; visual sphere radius=0.3
- added link rear_right_wheel, mass 2; collision sphere radius=0.3; visual sphere radius=0.3
Joints:
- added joint rear_left_wheel_joint: type continuous, parent chassis, child rear_left_wheel, origin xyz=-0.554283 0.625029 0.3 rpy=-1.5707 0 0, axis 0 0 1
- added joint rear_right_wheel_joint: type continuous, parent chassis, child rear_right_wheel, origin xyz=-0.554283 -0.625029 0.3 rpy=-1.5707 0 0, axis 0 0 1
