Commit message: Fix ros controller loading timeout

File: akm_500_display/urdf/mini_4wd_robot.urdf (robot description, URDF)
Before this commit: robot mini_4wd_robot, 8 links, 7 joints
Links:
- link lb_wheel_link: geometry collision cylinder length=0.02 radius=0.03; visual mesh filename=package://akm_500_display/meshes/mini_4wd_robot_meshes/lb_w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
- link lf_wheel_link: geometry collision cylinder length=0.02 radius=0.03; visual mesh filename=package://akm_500_display/meshes/mini_4wd_robot_meshes/lf_w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
- link rb_wheel_link: geometry collision cylinder length=0.02 radius=0.03; visual mesh filename=package://akm_500_display/meshes/mini_4wd_robot_meshes/rb_w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
- link rf_wheel_link: geometry collision cylinder length=0.02 radius=0.03; visual mesh filename=package://akm_500_display/meshes/mini_4wd_robot_meshes/rf_w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
