Commit message: Update akm_500_display to wheeltec_robot_display

File: wheeltec_robot_display/urdf/akm_base.xacro (robot description, xacro)
@@ -33,5 +33,5 @@
       <geometry>
         <mesh
-          filename="package://akm_500_display/meshes/V550_akm_robot_meshes/base_link.STL" />
+          filename="package://wheeltec_robot_display/meshes/V550_akm_robot_meshes/base_link.STL" />
       </geometry>
       <material
@@ -47,5 +47,5 @@
       <geometry>
         <mesh
-          filename="package://akm_500_display/meshes/V550_akm_robot_meshes/base_link.STL" />
+          filename="package://wheeltec_robot_display/meshes/V550_akm_robot_meshes/base_link.STL" />
       </geometry>
     </collision>
@@ -73,5 +73,5 @@
       <geometry>
         <mesh
-          filename="package://akm_500_display/meshes/V550_akm_robot_meshes/laser_link.STL" />
+          filename="package://wheeltec_robot_display/meshes/V550_akm_robot_meshes/laser_link.STL" />
       </geometry>
       <material
@@ -87,5 +87,5 @@
       <geometry>
         <mesh
-          filename="package://akm_500_display/meshes/V550_akm_robot_meshes/laser_link.STL" />
+          filename="package://wheeltec_robot_display/meshes/V550_akm_robot_meshes/laser_link.STL" />
       </geometry>
     </collision>
@@ -126,5 +126,5 @@
       <geometry>
         <mesh
-          filename="package://akm_500_display/meshes/V550_akm_robot_meshes/camera_link.STL" />
+          filename="package://wheeltec_robot_display/meshes/V550_akm_robot_meshes/camera_link.STL" />
       </geometry>
       <material
@@ -140,5 +140,5 @@
       <geometry>
         <mesh
-          filename="package://akm_500_display/meshes/V550_akm_robot_meshes/camera_link.STL" />
+          filename="package://wheeltec_robot_display/meshes/V550_akm_robot_meshes/camera_link.STL" />
       </geometry>
     </collision>
@@ -179,5 +179,5 @@
       <geometry>
         <mesh
-          filename="package://akm_500_display/meshes/V550_akm_robot_meshes/controller_link.STL" />
+          filename="package://wheeltec_robot_display/meshes/V550_akm_robot_meshes/controller_link.STL" />
       </geometry>
       <material
@@ -193,5 +193,5 @@
       <geometry>
         <mesh
-          filename="package://akm_500_display/meshes/V550_akm_robot_meshes/controller_link.STL" />
+          filename="package://wheeltec_robot_display/meshes/V550_akm_robot_meshes/controller_link.STL" />
       </geometry>
     </collision>
@@ -232,5 +232,5 @@
       <geometry>
         <mesh
-          filename="package://akm_500_display/meshes/V550_akm_robot_meshes/lb_wheel_link.STL" />
+          filename="package://wheeltec_robot_display/meshes/V550_akm_robot_meshes/lb_wheel_link.STL" />
       </geometry>
       <material
@@ -246,5 +246,5 @@
       <geometry>
         <mesh
-          filename="package://akm_500_display/meshes/V550_akm_robot_meshes/lb_wheel_link.STL" />
+          filename="package://wheeltec_robot_display/meshes/V550_akm_robot_meshes/lb_wheel_link.STL" />
       </geometry>
     </collision>
@@ -285,5 +285,5 @@
       <geometry>
         <mesh
-          filename="package://akm_500_display/meshes/V550_akm_robot_meshes/lf_wheel_link.STL" />
+          filename="package://wheeltec_robot_display/meshes/V550_akm_robot_meshes/lf_wheel_link.STL" />
       </geometry>
       <material
@@ -299,5 +299,5 @@
       <geometry>
         <mesh
-          filename="package://akm_500_display/meshes/V550_akm_robot_meshes/lf_wheel_link.STL" />
+          filename="package://wheeltec_robot_display/meshes/V550_akm_robot_meshes/lf_wheel_link.STL" />
       </geometry>
     </collision>
@@ -338,5 +338,5 @@
       <geometry>
         <mesh
-          filename="package://akm_500_display/meshes/V550_akm_robot_meshes/rb_wheel_link.STL" />
+          filename="package://wheeltec_robot_display/meshes/V550_akm_robot_meshes/rb_wheel_link.STL" />
       </geometry>
       <material
@@ -352,5 +352,5 @@
       <geometry>
         <mesh
-          filename="package://akm_500_display/meshes/V550_akm_robot_meshes/rb_wheel_link.STL" />
+          filename="package://wheeltec_robot_display/meshes/V550_akm_robot_meshes/rb_wheel_link.STL" />
       </geometry>
     </collision>
@@ -391,5 +391,5 @@
       <geometry>
         <mesh
-          filename="package://akm_500_display/meshes/V550_akm_robot_meshes/rf_wheel_link.STL" />
+          filename="package://wheeltec_robot_display/meshes/V550_akm_robot_meshes/rf_wheel_link.STL" />
       </geometry>
       <material
@@ -405,5 +405,5 @@
       <geometry>
         <mesh
-          filename="package://akm_500_display/meshes/V550_akm_robot_meshes/rf_wheel_link.STL" />
+          filename="package://wheeltec_robot_display/meshes/V550_akm_robot_meshes/rf_wheel_link.STL" />
       </geometry>
     </collision>

File: wheeltec_robot_display/urdf/mini_4wd_robot.urdf (robot description, URDF)
Before this commit: robot mini_4wd_robot, 8 links, 7 joints
Links:
- link base_link: geometry collision mesh filename=package://wheeltec_robot_display/meshes/mini_4wd_robot_mesh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; visual mesh filename=package://wheeltec_robot_display/meshes/mini_4wd_robot_mesh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
- link camera_link: geometry collision mesh filename=package://wheeltec_robot_display/meshes/mini_4wd_robot_mesh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; visual mesh filename=package://wheeltec_robot_display/meshes/mini_4wd_robot_mesh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
- link controller_link: geometry collision mesh filename=package://wheeltec_robot_display/meshes/mini_4wd_robot_mesh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; visual mesh filename=package://wheeltec_robot_display/meshes/mini_4wd_robot_mesh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
- link laser_link: geometry collision mesh filename=package://wheeltec_robot_display/meshes/mini_4wd_robot_mesh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; visual mesh filename=package://wheeltec_robot_display/meshes/mini_4wd_robot_mesh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
- link lb_wheel_link: geometry collision cylinder length=0.02 radius=0.03; visual mesh filename=package://wheeltec_robot_display/meshes/mini_4wd_robot_mesh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
- link lf_wheel_link: geometry collision cylinder length=0.02 radius=0.03; visual mesh filename=package://wheeltec_robot_display/meshes/mini_4wd_robot_mesh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
- link rb_wheel_link: geometry collision cylinder length=0.02 radius=0.03; visual mesh filename=package://wheeltec_robot_display/meshes/mini_4wd_robot_mesh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
- link rf_wheel_link: geometry collision cylinder length=0.02 radius=0.03; visual mesh filename=package://wheeltec_robot_display/meshes/mini_4wd_robot_mesh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
